File: solder.kicad_pcb (KiCad board)
At the start: 2 copper layers, 100.8 x 93.1 mm, 19 parts, among them M1 Motor_DC, SW2 SW_Push, SW3 SW_Push, SW4 SW_Push

Commit message: aaa
Parts:
- added G***: LOGO, LOGO, B.Cu at (221.1, 85.7)
- added G***: LOGO, LOGO, B.Cu at (192.0, 95.2)
- added G***: LOGO, LOGO, B.Cu at (179.2, 57.6)
- added G***: LOGO, LOGO, B.Cu at (193.0, 44.4)
- added G***: LOGO, LOGO, B.Cu at (219.5, 44.9)
- added G***: LOGO, LOGO, B.Cu at (231.6, 49.9)
- added G***: LOGO, LOGO, B.Cu at (196.4, 82.5)
- added G***: LOGO, LOGO, B.Cu at (180.8, 95.2)
- added G***: LOGO, LOGO, B.Cu at (180.2, 44.9)
- added G***: LOGO, LOGO, B.Cu at (208.9, 58.0)
- added G***: LOGO, LOGO, B.Cu at (205.9, 43.5)
- added G***: LOGO, LOGO, B.Cu at (203.3, 105.3)
- added G***: LOGO, LOGO, B.Cu at (160.7, 86.5)
- added G***: LOGO, LOGO, B.Cu at (208.4, 80.9)
- added G***: LOGO, LOGO, B.Cu at (174.0, 69.9)
- added G***: LOGO, LOGO, B.Cu at (169.8, 95.5)
- added G***: LOGO, LOGO, B.Cu at (145.7, 65.6)
- added G***: LOGO, LOGO, B.Cu at (190.9, 107.0)
- added G***: LOGO, LOGO, B.Cu at (202.5, 68.2)
- added G***: LOGO, LOGO, B.Cu at (179.0, 106.6)
- added G***: LOGO, LOGO, B.Cu at (198.3, 28.8)
- added G***: LOGO, LOGO, B.Cu at (222.7, 58.4)
- added G***: LOGO, LOGO, B.Cu at (216.3, 98.3)
- added G***: LOGO, LOGO, B.Cu at (153.3, 96.1)
- added G***: LOGO, LOGO, B.Cu at (170.9, 81.9)
- added G***: LOGO, LOGO, B.Cu at (212.2, 32.2)
- added G***: LOGO, LOGO, B.Cu at (185.7, 32.2)
- added G***: LOGO, LOGO, B.Cu at (158.1, 72.8)
- added G***: LOGO, LOGO, B.Cu at (166.5, 106.8)
- added G***: LOGO, LOGO, B.Cu at (188.5, 70.1)
- added G***: LOGO, LOGO, B.Cu at (216.9, 72.5)
- added G***: LOGO, LOGO, B.Cu at (183.0, 83.1)
- added G***: LOGO, LOGO, B.Cu at (194.4, 57.7)
- added G***: LOGO, LOGO, B.Cu at (147.0, 81.9)
- added G***: LOGO, LOGO, B.Cu at (205.3, 92.2)
- added H1: MountingHole, MountingHole:MountingHole_5mm, F.Cu at (178.5, 36.0)
- added Q1: BC107, Package_TO_SOT_THT:TO-18-3, F.Cu at (196.8, 49.1)
- added R1: R, Resistor_THT:R_Axial_DIN0207_L6.3mm_D2.5mm_P7.62mm_Horizontal, F.Cu at (203.9, 33.9)
Connections:
- D6 pad 2: Net-(D6-A) -> Net-(BT1-+)
- R6 pad 2: Net-(BT1--) -> Net-(Q1-C)
- R8 pad 1: Net-(BT1-+) -> Net-(Q1-B)
- R8 pad 2: Net-(D6-A) -> Net-(BT1--)
Routing:
- net Net-(Q1-B): track 0.00 -> 25.5 mm
- net Net-(BT1--): track 172.2 -> 195.3 mm
- net Net-(BT1-+): track 171.9 -> 194.5 mm
- net Net-(D6-A): track 18.8 -> 0.00 mm
- net Net-(Q1-C): track 0.00 -> 12.6 mm
- net Net-(D6-K): track 35.6 -> 24.7 mm
