File: solder.kicad_sch (KiCad schematic)
At the start: 18 parts, among them M1 Motor_DC, SW2 SW_Push, SW3 SW_Push, SW4 SW_Push

Commit message: aaa
Parts:
- added H1: MountingHole, MountingHole:MountingHole_5mm, symbol Mechanical:MountingHole
- added Q1: BC107, Package_TO_SOT_THT:TO-18-3, symbol Transistor_BJT:BC107
- added R1: R, Resistor_THT:R_Axial_DIN0207_L6.3mm_D2.5mm_P7.62mm_Horizontal, symbol Device:R
Connections:
- net at BT1.2 (-), M1.2 (-), R2.2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: now also R8.2, Q1.1 (E); no longer R6.2
- net at BT1.1 (+), RV1.1, RV2.1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: now also D6.2 (A), R1.1; no longer R8.1
- new net: Q1.2 (B), R1.2, R8.1
- new net: Q1.3 (C), R6.2
Other:
- moved on the sheet: D6, M1, R6, R8, RV2
